Commit message: launch webots and spawn a robot

File: src/magni_description/urdf/magni.urdf.xacro (robot description, xacro)
@@ -27,5 +27,5 @@
       </geometry>
     </visual>
-	<visual>
+	  <visual>
       <origin xyz="${-wheel_xpos-0.169} 0.17 ${-wheel_r+0.09}" rpy="0 0 ${pi}" />
       <geometry>
@@ -33,5 +33,5 @@
       </geometry>
     </visual>
-	<visual>
+	  <visual>
       <origin xyz="${-wheel_xpos-0.169} -0.17 ${-wheel_r+0.09}" rpy="0 0 ${pi}" />
       <geometry>
@@ -40,8 +40,8 @@
     </visual>
     <collision>
-	  <origin xyz="${-wheel_xpos} 0 ${-wheel_r+0.151}" rpy="0 0 0" />
-      <geometry>
-        <box size="0.398 0.268 0.160"/>
-      </geometry>
+	    <origin xyz="${-wheel_xpos} 0 ${-wheel_r+0.151}" rpy="0 0 0" />
+        <geometry>
+          <box size="0.398 0.268 0.160"/>
+        </geometry>
     </collision>
     <collision>
@@ -130,6 +130,6 @@
   <link name="base_footprint"/>
   <joint name="base_footprint_joint" type="fixed">
-    <parent link="base_footprint"/>
-    <child link="base_link"/>
+    <parent link="base_link"/>
+    <child link="base_footprint"/>
     <origin xyz="0 0 ${wheel_r}" rpy="0 0 0"/>
   </joint>

Commit message: fixing dev container

File: src/magni_description/urdf/magni.urdf.xacro (robot description, xacro)
@@ -178,5 +178,5 @@
       </collision>
     </link>
-    <joint name="${prefix}_caster_wheel_joint" type="fixed">
+    <joint name="${prefix}_caster_wheel_joint" type="continuous">
       <parent link="base_link"/>
       <child link="${prefix}_caster_wheel"/>

Commit message: add raspberry pi cam simulation

File: src/magni_description/urdf/magni.urdf.xacro (robot description, xacro)
@@ -1,5 +1,5 @@
 <?xml version="1.0"?>
 <robot xmlns:xacro="http://www.ros.org/wiki/xacro" name="magni">
-  <xacro:arg name="sonars_installed" default="true"/>
+  <xacro:arg name="sonars_installed" default="false"/>
   <xacro:property name="sonars_installed" value="$(arg sonars_installed)"/>
   <xacro:arg name="shell_installed" default="false"/>
@@ -7,7 +7,7 @@
   <xacro:arg name="tower_installed" default="false"/>
   <xacro:property name="tower_installed" value="$(arg tower_installed)"/>
-  <xacro:arg name="camera_extrinsics_file" default=""/>
+  <xacro:arg name="camera_extrinsics_file" default="extrinsics/camera_extrinsics_forward.yaml"/>
   <xacro:property name="camera_extrinsics_file" value="$(arg camera_extrinsics_file)"/>
-  <xacro:arg name="lidar_extrinsics_file" default=""/>
+  <xacro:arg name="lidar_extrinsics_file" default="extrinsics/lidar_extrinsics_top_plate_center.yaml"/>
   <xacro:property name="lidar_extrinsics_file" value="$(arg lidar_extrinsics_file)"/>
   <xacro:property name="wheel_r" value="0.1" />

File: src/magni_description/urdf/sensors/raspi_camera.xacro (robot description, xacro)
@@ -17,7 +17,7 @@
       </visual>
       <collision>
-        <origin xyz="0 0 0" rpy="0 0 ${pi/2}" />
+        <origin xyz="0 0 0" rpy="0 0 0" />
         <geometry>
-          <box size="0.03 0.026 0.016"/>
+          <box size="0.016 0.026 0.03"/>
         </geometry>
       </collision>
@@ -30,8 +30,6 @@
       <origin xyz="0.005 0 0" rpy="${-pi/2} 0 ${-pi/2}" />
     </joint>
-    <!-- Gazebo sensor plugin. Gazebo sensor is attached to camera link (${name}) but publishes its messages to ${name}_sensor frame. -->
-    <gazebo reference="${name}">
+    <gazebo reference="${name}_sensor">
       <sensor type="camera" name="camera1">
-        <visualize>false</visualize>
         <update_rate>30.0</update_rate>
         <camera name="raspi_camera">
@@ -47,19 +45,4 @@
           </clip>
         </camera>
-        <!-- Gazebo-ROS interface plugin -->
-        <plugin name="camera_controller" filename="libgazebo_ros_camera.so">
-          <alwaysOn>true</alwaysOn>
-          <updateRate>0.0</updateRate>
-          <cameraName></cameraName>
-          <imageTopicName>${name}_node/image</imageTopicName>
-          <cameraInfoTopicName>${name}_node/camera_info</cameraInfoTopicName>
-          <frameName>${name}_sensor</frameName>
-          <hackBaseline>0.07</hackBaseline>
-          <distortionK1>0.0</distortionK1>
-          <distortionK2>0.0</distortionK2>
-          <distortionK3>0.0</distortionK3>
-          <distortionT1>0.0</distortionT1>
-          <distortionT2>0.0</distortionT2>
-        </plugin>
       </sensor>
     </gazebo>

File: src/magni_webots/resource/magni_wb.urdf.xacro (robot description, xacro)
@@ -2,4 +2,10 @@
 <robot name="magni" xmlns:xacro="http://wiki.ros.org/xacro">
     <webots>
+        <device reference="camera1" type="Camera">
+            <ros>
+                <topicName>/rpicam</topicName>
+                <alwaysOn>true</alwaysOn>
+            </ros>
+        </device>
         <plugin type="magni_driver::MagniDriver" />
     </webots>
